File: larsskj-014.kicad_sch (KiCad schematic)
At the start: 6 parts, among them J1 Conn_01x01_Pin, J2 Conn_01x01_Pin, J3 Conn_01x01_Pin, J4 Conn_01x01_Pin, J5 Conn_01x01_Pin, J6 Conn_01x01_Pin

Commit message: Update metadata.
Other:
- company: (none) -> Lars Skjærlund
- title: (none) -> larsskj-014
Changed lines of the file:
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@@
 	(generator_version "9.0")
 	(paper "A4")
+	(title_block
+		(title "larsskj-014")
+		(date "2025-10-06")
+		(rev "01")
+		(company "Lars Skjærlund")
+		(comment 4 "A board to provide power to scale models using pogo pins.")
+	)
 	(junction
 		(at 140.97 96.52)

Commit message: Ready for revision #2
Parts:
- J3, J4: LCSC (none) -> C5157269
Changed lines of the file:
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@@
+			)
+		)
+		(property "LCSC" "C5157269"
+			(at 160.02 101.6 0)
+			(effects
+				(font
+					(size 1.27 1.27)
+				)
+				(hide yes)
 			)
 		)
@@
 			(at 160.02 96.52 0)
 			(effects
+				(font
+					(size 1.27 1.27)
+				)
+				(hide yes)
+			)
+		)
+		(property "LCSC" "C5157269"
+			(at 160.02 96.52 0)
+			(effects
